File: pcb/leds.kicad_sch (KiCad schematic)
At the start: 46 parts, among them Q1 NPN, U10 SK6812MINI-FA, U11 SK6812MINI-FA, U12 SK6812MINI-FA, U13 SK6812MINI-FA, U14 SK6812MINI-FA, U15 SK6812MINI-FA, U16 SK6812MINI-FA, U17 SK6812MINI-FA, U18 SK6812MINI-FA, U19 SK6812MINI-FA, U2 SK6812MINI-FA, U20 SK6812MINI-FA, U21 SK6812MINI-FA, U3 SK6812MINI-FA, U4 SK6812MINI-FA, U5 SK6812MINI-FA, U6 SK6812MINI-FA, U7 SK6812MINI-FA, U8 SK6812MINI-FA, U9 SK6812MINI-FA

Commit message: Finished schematic
Parts:
- removed Q1: NPN, symbol Simulation_SPICE:NPN
- removed R4, R5: 10kR, symbol Device:R
- added U14: SN74LV1T34DCKR_C48543212, lcsc_lib:SC-70-5_L2.1-W1.3-P0.65-LS2.1-BR, symbol lcsc:SN74LV1T34DCKR_C48543212
- C17: renamed from C5; footprint (none) -> Capacitor_SMD:C_0603_1608Metric; LCSC Part (none) -> C14663
- C18: renamed from C6; footprint (none) -> Capacitor_SMD:C_0603_1608Metric; LCSC Part (none) -> C14663
- C19: renamed from C7; footprint (none) -> Capacitor_SMD:C_0603_1608Metric; LCSC Part (none) -> C14663
- C20: renamed from C8; footprint (none) -> Capacitor_SMD:C_1210_3225Metric; LCSC Part (none) -> C7432790
- C21: renamed from C9; footprint (none) -> Capacitor_SMD:C_0603_1608Metric; LCSC Part (none) -> C14663
- C22: renamed from C10; footprint (none) -> Capacitor_SMD:C_0603_1608Metric; LCSC Part (none) -> C14663
- C23: renamed from C11; footprint (none) -> Capacitor_SMD:C_0603_1608Metric; LCSC Part (none) -> C14663
- C24: renamed from C12; footprint (none) -> Capacitor_SMD:C_0603_1608Metric; LCSC Part (none) -> C14663
- C25: renamed from C13; footprint (none) -> Capacitor_SMD:C_0603_1608Metric; LCSC Part (none) -> C14663
- C26: renamed from C14; footprint (none) -> Capacitor_SMD:C_0603_1608Metric; LCSC Part (none) -> C14663
- C27: renamed from C15; footprint (none) -> Capacitor_SMD:C_0603_1608Metric; LCSC Part (none) -> C14663
- C28: renamed from C16; footprint (none) -> Capacitor_SMD:C_0603_1608Metric; LCSC Part (none) -> C14663
- C29: renamed from C17; footprint (none) -> Capacitor_SMD:C_0603_1608Metric; LCSC Part (none) -> C14663
- C30: renamed from C18; footprint (none) -> Capacitor_SMD:C_0603_1608Metric; LCSC Part (none) -> C14663
- C31: renamed from C19; footprint (none) -> Capacitor_SMD:C_0603_1608Metric; LCSC Part (none) -> C14663
- C32: renamed from C20; footprint (none) -> Capacitor_SMD:C_0603_1608Metric; LCSC Part (none) -> C14663
- C33: renamed from C21; footprint (none) -> Capacitor_SMD:C_0603_1608Metric; LCSC Part (none) -> C14663
- C34: renamed from C22; footprint (none) -> Capacitor_SMD:C_0603_1608Metric; LCSC Part (none) -> C14663
- C35: renamed from C23; footprint (none) -> Capacitor_SMD:C_0603_1608Metric; LCSC Part (none) -> C14663
- C36: renamed from C24; footprint (none) -> Capacitor_SMD:C_0603_1608Metric; LCSC Part (none) -> C14663
- C37: renamed from C25; footprint (none) -> Capacitor_SMD:C_0603_1608Metric; LCSC Part (none) -> C14663
- R14: renamed from R6; value 510 -> 510R; footprint (none) -> Resistor_SMD:R_0603_1608Metric; LCSC Part (none) -> C2907179
- R15: renamed from R7; value 510 -> 510R; footprint (none) -> Resistor_SMD:R_0603_1608Metric; LCSC Part (none) -> C2907179
- renumbered U2 to U11, U3 to U12, U4 to U13, U5 to U15, U6 to U16, U7 to U17, U8 to U18, U9 to U19, U10 to U20, U11 to U21, U12 to U22, U13 to U23, U14 to U24, U15 to U25, U16 to U26, U17 to U27, U18 to U28, U19 to U29, U20 to U30, U21 to U31
Connections:
- net +5V: now also U14.5 (VCC)
- net GND: now also U14.3 (GND)
- net at R14.1: now also U14.4 (Y)
- new net DIN: U14.2 (A)
- no-connect marks 0 -> 2
