File: pcb/power.kicad_sch (KiCad schematic)
At the start: 35 parts, among them SW4 SKRPACE010, U27 BQ24073RGTR, U28 LP5907MFX-3.3/NOPB, U29 TPS62237DRYR, U30 TPS61023DRLR

Commit message: Finished schematic
Parts:
- removed C40, C41: 22uF, symbol Device:C
- removed D5, D6: BAT54X, lcsc_lib:SOD-523_L1.2-W0.8-LS1.6-RD, symbol lcsc:BAT54X_C51315114
- removed R13, R14: 1kR, symbol Device:R
- added C43: 1uF, Capacitor_SMD:C_0603_1608Metric, symbol Device:C
- added C47, C48: 22uF, Capacitor_SMD:C_0603_1608Metric, symbol Device:C
- added R19, R21: 10kR, Resistor_SMD:R_0603_1608Metric, symbol Device:R
- added R23: 100kR, Resistor_SMD:R_0603_1608Metric, symbol Device:R
- added U35: TPS3840DL35DBVR, lcsc_lib:SOT-23-5_L2.9-W1.6-P0.95-LS2.8-BR, symbol lcsc:TPS3840DL35DBVR
- C38: renamed from C35; footprint (none) -> Capacitor_SMD:C_0603_1608Metric; LCSC Part (none) -> C19702
- C39: renamed from C34; footprint (none) -> Capacitor_SMD:C_0603_1608Metric; LCSC Part (none) -> C19666
- C40: renamed from C38; value C -> 2.2uF; footprint (none) -> Capacitor_SMD:C_0805_2012Metric; LCSC Part (none) -> C19110
- C41: renamed from C37; value C -> 4.7uF; footprint (none) -> Capacitor_SMD:C_0603_1608Metric; LCSC Part (none) -> C19666
- C42: renamed from C32; footprint (none) -> Capacitor_SMD:C_0603_1608Metric; LCSC Part (none) -> C19666
- C44: renamed from C33; footprint (none) -> Capacitor_SMD:C_0603_1608Metric; LCSC Part (none) -> C19702
- C45: renamed from C36; footprint (none) -> Capacitor_SMD:C_0603_1608Metric; LCSC Part (none) -> C19702
- C46: renamed from C39; footprint (none) -> Capacitor_SMD:C_0603_1608Metric; LCSC Part (none) -> C96446
- L3: renamed from L2; value L -> 1uH; footprint (none) -> Inductor_SMD:L_1008_2520Metric; LCSC Part (none) -> C5179444
- L4: renamed from L3; footprint (none) -> Inductor_SMD:L_1008_2520Metric; LCSC Part (none) -> C5179444
- R16: renamed from R15; footprint (none) -> Resistor_SMD:R_0603_1608Metric; LCSC Part (none) -> C2907081
- R17: renamed from R16; footprint (none) -> Resistor_SMD:R_0603_1608Metric; LCSC Part (none) -> C2998107
- R18: renamed from R12; footprint (none) -> Resistor_SMD:R_0603_1608Metric; LCSC Part (none) -> C2930027
- R20: renamed from R18; footprint (none) -> Resistor_SMD:R_0603_1608Metric; LCSC Part (none) -> C2906980
- R22: renamed from R17; value 10kR -> 100kR; footprint (none) -> Resistor_SMD:R_0603_1608Metric; LCSC Part (none) -> C2906980
- R24: renamed from R21; footprint (none) -> Resistor_SMD:R_0603_1608Metric; LCSC Part (none) -> C2849083
- R25: renamed from R19; value 10kR -> 100kR; footprint (none) -> Resistor_SMD:R_0603_1608Metric; LCSC Part (none) -> C2906980
- R26: renamed from R20; footprint (none) -> Resistor_SMD:R_0603_1608Metric; LCSC Part (none) -> C2906980
- TP6: footprint (none) -> TestPoint:TestPoint_Loop_D2.50mm_Drill1.0mm
- TP7: renamed from TP5; footprint (none) -> TestPoint:TestPoint_Loop_D2.50mm_Drill1.0mm
- TP8: renamed from TP4; footprint (none) -> TestPoint:TestPoint_Loop_D2.50mm_Drill1.0mm
- TP9: renamed from TP3; footprint (none) -> TestPoint:TestPoint_Loop_D2.50mm_Drill1.0mm
- renumbered D3 to D1, D4 to D2, U29 to U32, U27 to U33, U28 to U34, U30 to U36
Connections:
- net CHG: now also U33.9 (~{CHG}), R19.1
- net GND: now also C43.2, C47.2, C48.2, R23.2, U35.3 (GND)
- net GNSS_EN: now also R23.1
- net LED_5V: now also R24.1, U36.6 (VOUT), C47.1, C48.1; no longer R24.2, R26.1, U36.1 (FB)
- net MAIN_EN: now also U35.1 (~{RESET})
- net PGOOD: now also U33.7 (~{PGOOD}), R21.1
- net VSYS: now also C43.1, R19.2, R21.2, U35.2 (VDD)
- new net: R24.2, R26.1, U36.1 (FB)
- no-connect marks 4 -> 6
Other:
- moved on the sheet: C44, D1, D2, R20, R22, R24, R26, SW4
